File: camera-detector-pcb/camera-detector-pcb.kicad_pcb (KiCad board)
At the start: 2 copper layers, 29 parts, among them J1 Conn_01x07, J2 Conn_01x07, J3 Conn_01x04, J8 Conn_01x01, J9 Conn_01x01, Q1 PN2222A, SW1 SW_Push, SW2 SW_Push, SW3 SW_Wuerth_450301014042, SW4 SW_Push, U1 74AHCT125

Commit message: final pcb
Parts:
- removed C3, C4: 100uf, Capacitor_THT:C_Radial_D5.0mm_H7.0mm_P2.00mm
- removed C5: 1000uf, Capacitor_THT:C_Radial_D8.0mm_H11.5mm_P3.50mm
- removed D2: 1N5819, Diode_THT:D_DO-41_SOD81_P10.16mm_Horizontal
- removed R10, R11, R2, R3, R4, R5, R8, R9: R, Resistor_THT:R_Axial_DIN0207_L6.3mm_D2.5mm_P15.24mm_Horizontal
- added J10: Conn_01x01, Connector_PinHeader_2.54mm:PinHeader_1x01_P2.54mm_Vertical, F.Cu at (139.2, 245.9)
- added J11: Conn_01x01, Connector_PinHeader_2.54mm:PinHeader_1x01_P2.54mm_Vertical, F.Cu at (139.2, 257.0)
- added J12: Conn_01x01, Connector_PinHeader_2.54mm:PinHeader_1x01_P2.54mm_Vertical, F.Cu at (139.2, 251.5)
- added J13: Conn_01x01, Connector_PinHeader_2.54mm:PinHeader_1x01_P2.54mm_Vertical, F.Cu at (151.9, 167.6)
- added J14: Conn_01x01, Connector_PinHeader_2.54mm:PinHeader_1x01_P2.54mm_Vertical, F.Cu at (146.8, 167.6)
- added J15: Conn_01x01, Connector_PinHeader_2.54mm:PinHeader_1x01_P2.54mm_Vertical, F.Cu at (157.0, 167.6)
- added J4: Conn_01x01, Connector_PinHeader_2.54mm:PinHeader_1x01_P2.54mm_Vertical, F.Cu at (174.2, 172.7)
- added J5: Conn_01x01, Connector_PinHeader_2.54mm:PinHeader_1x01_P2.54mm_Vertical, F.Cu at (174.0, 188.0)
- added J6: Conn_01x01, Connector_PinHeader_2.54mm:PinHeader_1x01_P2.54mm_Vertical, F.Cu at (174.2, 167.6)
- added J7: Conn_01x01, Connector_PinHeader_2.54mm:PinHeader_1x01_P2.54mm_Vertical, F.Cu at (174.0, 182.9)
- added REF**: MountingHole_3.2mm_M3_ISO7380, MountingHole:MountingHole_3.2mm_M3_ISO7380, F.Cu at (177.8, 203.2)
- added REF**: MountingHole_3.2mm_M3_ISO7380, MountingHole:MountingHole_3.2mm_M3_ISO7380, F.Cu at (127.0, 157.5)
- added REF**: MountingHole_3.2mm_M3_ISO7380, MountingHole:MountingHole_3.2mm_M3_ISO7380, F.Cu at (127.0, 264.2)
- added REF**: MountingHole_3.2mm_M3_ISO7380, MountingHole:MountingHole_3.2mm_M3_ISO7380, F.Cu at (177.8, 232.7)
- added REF**: MountingHole_3.2mm_M3_ISO7380, MountingHole:MountingHole_3.2mm_M3_ISO7380, F.Cu at (127.0, 209.3)
- C1: footprint Capacitor_THT:C_Disc_D4.7mm_W2.5mm_P5.00mm -> Capacitor_THT:C_Disc_D3.0mm_W1.6mm_P2.50mm
- C2: value 10uf -> 1000uf; footprint Capacitor_THT:C_Radial_D8.0mm_H7.0mm_P3.50mm -> Capacitor_THT:CP_Radial_D10.0mm_P5.00mm
- Q1: footprint Package_TO_SOT_THT:TO-92_Inline -> Package_TO_SOT_THT:TO-92_Inline_Wide
- R6: value R -> 1k; footprint Resistor_THT:R_Axial_DIN0207_L6.3mm_D2.5mm_P15.24mm_Horizontal -> Resistor_THT:R_Axial_DIN0204_L3.6mm_D1.6mm_P5.08mm_Horizontal
- R7: value R -> 330; footprint Resistor_THT:R_Axial_DIN0207_L6.3mm_D2.5mm_P15.24mm_Horizontal -> Resistor_THT:R_Axial_DIN0204_L3.6mm_D1.6mm_P5.08mm_Horizontal
- U1: footprint Package_DIP:DIP-14_W7.62mm -> Package_DIP:CERDIP-14_W7.62mm_SideBrazed
- moved BZ1 191.9 mm to (173.2, 263.6), turned to 90 degrees
- moved R6 189.8 mm to (163.6, 264.7), turned to 90 degrees
- moved J2 172.3 mm to (159.5, 264.4), turned to 180 degrees
- moved SW1 167.1 mm to (148.6, 234.5)
- moved J1 155.2 mm to (144.3, 249.2)
- moved Q1 150.0 mm to (165.2, 246.4), turned to -90 degrees
- moved SW2 147.6 mm to (148.6, 223.1)
- moved C2 141.0 mm to (141.2, 230.8), turned to -90 degrees
- moved D1 139.5 mm to (164.6, 240.8), turned to 90 degrees
- moved U1 135.3 mm to (142.5, 221.5), turned to 180 degrees
- moved SW4 127.9 mm to (148.6, 211.4)
- moved SW3 122.7 mm to (170.2, 215.9), turned to 90 degrees
- moved C1 119.6 mm to (134.9, 226.6)
- moved R7 112.6 mm to (144.8, 193.0), turned to 90 degrees
- moved J9 109.1 mm to (164.6, 215.9), turned to -90 degrees
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Connections:
- net /3.3V renamed 3.3V
- net /D2 renamed D2
- net /D3 renamed D3
- net /D4 renamed D4
- net /D5 renamed D5
- net /D6 renamed D6
- net /D8 renamed D8
- BZ1 pad 1: unconnected-(BZ1-+-Pad1) -> 5V
- BZ1 pad 2: unconnected-(BZ1---Pad2) -> Net-(BZ1--)
- C1 pad 1: unconnected-(C1-Pad1) -> 5V
- C1 pad 2: unconnected-(C1-Pad2) -> GND
- C2 pad 1: unconnected-(C2-Pad1) -> 5V
- C2 pad 2: unconnected-(C2-Pad2) -> GND
- D1 pad 1: unconnected-(D1-K-Pad1) -> 5V
- D1 pad 2: unconnected-(D1-A-Pad2) -> Net-(BZ1--)
- J1 pad 1: /D0 -> D0
- J1 pad 2: /D1 -> D1
- J2 pad 1: /D7 -> D7
- J2 pad 3: /D9 -> D9
- J2 pad 4: /D10 -> D10
- J2 pad 7: VBAT -> unconnected-(J2-Pin_7-Pad7)
- Q1 pad 1: unconnected-(Q1-E-Pad1) -> GND
- Q1 pad 2: unconnected-(Q1-B-Pad2) -> Net-(Q1-B)
- Q1 pad 3: unconnected-(Q1-C-Pad3) -> Net-(BZ1--)
- R6 pad 1: unconnected-(R6-Pad1) -> D10
- R6 pad 2: unconnected-(R6-Pad2) -> Net-(Q1-B)
- R7 pad 1: unconnected-(R7-Pad1) -> Net-(R7-Pad1)
- R7 pad 2: unconnected-(R7-Pad2) -> /DIN
- SW1 pad 1: /D9 -> D7
- SW4 pad 1: /D7 -> D9
- U1 pad 1: unconnected-(U1-Pad1) -> GND
- U1 pad 14: (no net) -> 5V
- U1 pad 2: unconnected-(U1-Pad2) -> D1
- U1 pad 3: unconnected-(U1-Pad3) -> Net-(R7-Pad1)
- U1 pad 7: (no net) -> GND
Routing:
- net 5V: track 0.00 -> 210.4 mm
- net D5: track 0.00 -> 88.8 mm
- net D4: track 0.00 -> 86.1 mm
- net 3.3V: track 0.00 -> 83.5 mm
- net D9: track 0.00 -> 53.9 mm
- net /IN+: track 0.00 -> 47.9 mm
- net D8: track 0.00 -> 43.6 mm
- net D1: track 0.00 -> 35.6 mm
- net Net-(BZ1--): track 0.00 -> 35.1 mm
- net D7: track 0.00 -> 34.3 mm
- net Net-(R7-Pad1): track 0.00 -> 25.6 mm
- net /DIN: track 0.00 -> 23.3 mm
- net Net-(Q1-B): track 0.00 -> 11.7 mm
- net D10: track 0.00 -> 9.55 mm
- net D0: track 0.00 -> 6.02 mm
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- added copper zone on F.Cu, net GND
Other:
- board outline added: 61 x 116.8 mm
- board text added: "led"
- board text added: "rf module"
